File: PCBs/StroomMeterACS712.kicad_sch (KiCad schematic)
At the start: 6 parts, among them J2 AC_Live, J3 AC_Live, Q1 BC547, U1 WeMos_D1_mini, U2 ACS712xLCTR-05B

Commit message: algemeen1
Parts:
- gave numbers to parts that had none: 1
Connections:
- net VCC: now also U1.9 (5V)
- net D0: now reaches U1.1 (~{RST})
- net D0: now also U1.3 (D0)
- net SDA: now reaches U1.13 (SDA/D2)
- net SCL: now reaches U1.14 (SCL/D1)
- net AC712: now reaches U1.2 (A0)
Other:
- note removed: "D0"

Commit message: labels bijgewerkt
Parts:
- J3: value AC_Live -> AC_Neutral
Connections:
- net AC712 is gone; now on net Data: U1.2 (A0)
- net GND: now also J1.4 (Pin_4)
- net SCL: now also J1.2 (Pin_2)
- net SDA: now also J1.1 (Pin_1)
- net VCC: now also J1.3 (Pin_3)
- net AC_L: now reaches J2.1 (Pin_1), U2.1 (IP+), U2.2 (IP+)
- net AC_N: now reaches J3.1 (Pin_1), U2.3 (IP-), U2.4 (IP-)
- net Data: now reaches U2.7 (VIOUT)
- net AanUit: now reaches Q1.2 (B)
- net AanUit: now also U1.12 (D3)
- net D0 renamed DpSlp
- no-connect marks 4 -> 9
Other:
- note removed: "AC712"
- note removed: "ACS"
- note removed: "AC_L"
- note removed: "GND"
- note removed: "Oled_128X32"
- note removed: "SCL"
- note removed: "SDA"
- note removed: "VCC"
Changed lines of the file:
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@@
     (date "2022-12-06")
   )
-  (no_connect (at 33.655 48.895))
-  (no_connect (at 33.655 46.355))
+  (no_connect (at 36.195 48.895))
+  (no_connect (at 36.195 46.355))
   (no_connect (at 48.895 28.575))
+  (no_connect (at 60.325 59.055))
+  (no_connect (at 60.325 48.895))
+  (no_connect (at 60.325 51.435))
+  (no_connect (at 60.325 53.975))
+  (no_connect (at 60.325 56.515))
   (no_connect (at 111.125 53.34))
-  (bus_entry (at 60.325 43.815) (size 2.54 2.54)
-    (stroke (width 0) (type default) (color 0 0 0 0))
-  )
-  (bus_entry (at 60.325 41.275) (size 2.54 2.54)
-    (stroke (width 0) (type default) (color 0 0 0 0))
-  )
-  (bus_entry (at 60.325 36.195) (size 2.54 2.54)
-    (stroke (width 0) (type default) (color 0 0 0 0))
-  )
-  (bus_entry (at 60.325 56.515) (size 2.54 2.54)
-    (stroke (width 0) (type default) (color 0 0 0 0))
-  )
-  (bus_entry (at 60.325 48.895) (size 2.54 2.54)
-    (stroke (width 0) (type default) (color 0 0 0 0))
-  )
-  (bus_entry (at 60.325 46.355) (size 2.54 2.54)
-    (stroke (width 0) (type default) (color 0 0 0 0))
-  )
-  (bus_entry (at 60.325 59.055) (size 2.54 2.54)
-    (stroke (width 0) (type default) (color 0 0 0 0))
-  )
-  (bus_entry (at 60.325 53.975) (size 2.54 2.54)
-    (stroke (width 0) (type default) (color 0 0 0 0))
-  )
-  (bus_entry (at 60.325 51.435) (size 2.54 2.54)
-    (stroke (width 0) (type default) (color 0 0 0 0))
-  )
-  (bus_entry (at 60.325 38.735) (size 2.54 2.54)
-    (stroke (width 0) (type default) (color 0 0 0 0))
-  )
   (bus_entry (at 71.12 77.47) (size 2.54 2.54)
     (stroke (width 0) (type default) (color 0 0 0 0))
@@
     (stroke (width 0) (type default) (color 0 0 0 0))
   )
-  (bus (pts (xy 62.865 51.435) (xy 62.865 53.975))
-    (stroke (width 0) (type default) (color 0 0 0 0))
-  )
   (wire (pts (xy 41.275 24.765) (xy 43.815 24.765))
     (stroke (width 0) (type default) (color 0 0 0 0))
   )
-  (bus (pts (xy 62.865 59.055) (xy 62.865 61.595))
-    (stroke (width 0) (type default) (color 0 0 0 0))
-  )
   (wire (pts (xy 56.515 48.895) (xy 60.325 48.895))
     (stroke (width 0) (type default) (color 0 0 0 0))
@@
     (stroke (width 0) (type default) (color 0 0 0 0))
   )
-  (bus (pts (xy 71.12 69.85) (xy 71.12 72.39))
-    (stroke (width 0) (type default) (color 0 0 0 0))
-  )
   (wire (pts (xy 56.515 53.975) (xy 60.325 53.975))
     (stroke (width 0) (type default) (color 0 0 0 0))
   )
-  (bus (pts (xy 62.865 46.355) (xy 62.865 48.895))
-    (stroke (width 0) (type default) (color 0 0 0 0))
-  )
-  (bus (pts (xy 71.12 64.135) (xy 71.12 69.85))
+  (wire (pts (xy 56.515 36.195) (xy 60.325 36.195))
     (stroke (width 0) (type default) (color 0 0 0 0))
   )
@@
     (stroke (width 0) (type default) (color 0 0 0 0))
   )
-  (bus (pts (xy 62.865 43.815) (xy 62.865 46.355))
-    (stroke (width 0) (type default) (color 0 0 0 0))
-  )
   (wire (pts (xy 73.66 72.39) (xy 76.835 72.39))
     (stroke (width 0) (type default) (color 0 0 0 0))
   )
-  (bus (pts (xy 62.865 41.275) (xy 62.865 43.815))
-    (stroke (width 0) (type default) (color 0 0 0 0))
-  )
-  (bus (pts (xy 71.12 74.93) (xy 71.12 77.47))
-    (stroke (width 0) (type default) (color 0 0 0 0))
-  )
   (wire (pts (xy 106.68 53.34) (xy 111.125 53.34))
     (stroke (width 0) (type default) (color 0 0 0 0))
   )
-  (bus (pts (xy 62.865 48.895) (xy 62.865 51.435))
-    (stroke (width 0) (type default) (color 0 0 0 0))
-  )
-  (bus (pts (xy 62.865 38.735) (xy 62.865 41.275))
-    (stroke (width 0) (type default) (color 0 0 0 0))
-  )
-  (wire (pts (xy 33.655 48.895) (xy 36.195 48.895))
+  (wire (pts (xy 43.815 24.765) (xy 43.815 28.575))
     (stroke (width 0) (type default) (color 0 0 0 0))
   )
@@
     (stroke (width 0) (type default) (color 0 0 0 0))
   )
-  (bus (pts (xy 62.865 53.975) (xy 62.865 56.515))
-    (stroke (width 0) (type default) (color 0 0 0 0))
-  )
-  (wire (pts (xy 33.655 46.355) (xy 36.195 46.355))
+  (wire (pts (xy 46.355 69.215) (xy 46.355 73.66))
+    (stroke (width 0) (type default) (color 0 0 0 0))
+  )
+  (wire (pts (xy 56.515 46.355) (xy 60.325 46.355))
     (stroke (width 0) (type default) (color 0 0 0 0))
   )
@@
     (stroke (width 0) (type default) (color 0 0 0 0))
   )
-  (bus (pts (xy 62.865 64.135) (xy 71.12 64.135))
-    (stroke (width 0) (type default) (color 0 0 0 0))
-  )
-  (wire (pts (xy 46.355 69.215) (xy 46.355 73.66))
-    (stroke (width 0) (type default) (color 0 0 0 0))
-  )
   (wire (pts (xy 56.515 38.735) (xy 60.325 38.735))
     (stroke (width 0) (type default) (color 0 0 0 0))
   )
-  (bus (pts (xy 62.865 61.595) (xy 62.865 64.135))
-    (stroke (width 0) (type default) (color 0 0 0 0))
-  )
-  (wire (pts (xy 56.515 46.355) (xy 60.325 46.355))
-    (stroke (width 0) (type default) (color 0 0 0 0))
-  )
-  (wire (pts (xy 56.515 36.195) (xy 60.325 36.195))
-    (stroke (width 0) (type default) (color 0 0 0 0))
-  )
-  (bus (pts (xy 71.12 72.39) (xy 71.12 74.93))
-    (stroke (width 0) (type default) (color 0 0 0 0))
-  )
-  (wire (pts (xy 43.815 28.575) (xy 43.815 24.765))
-    (stroke (width 0) (type default) (color 0 0 0 0))
-  )
   (wire (pts (xy 56.515 43.815) (xy 60.325 43.815))
     (stroke (width 0) (type default) (color 0 0 0 0))
   )
-  (bus (pts (xy 62.865 56.515) (xy 62.865 59.055))
-    (stroke (width 0) (type default) (color 0 0 0 0))
-  )
-  (text "GND" (at 74.295 80.01 0)
-    (effects (font (size 0.67 0.67)) (justify left bottom))
-  )
-  (text "SCL" (at 74.295 74.93 0)
-    (effects (font (size 0.67 0.67)) (justify left bottom))
-  )
-  (text "VCC" (at 74.295 77.47 0)
-    (effects (font (size 0.67 0.67)) (justify left bottom))
-  )
-  (text "ACS" (at 86.995 27.94 0)
-    (effects (font (size 0.55 0.55)) (justify left bottom))
-  )
-  (text "GND" (at 96.52 60.96 270)
-    (effects (font (size 0.67 0.67)) (justify right bottom))
-  )
-  (text "GND" (at 46.355 71.12 270)
-    (effects (font (size 0.67 0.67)) (justify right bottom))
-  )
-  (text "Oled_128X32" (at 64.135 44.45 270)
-    (effects (font (size 0.55 0.55)) (justify right bottom))
-  )
-  (text "AC_L" (at 83.82 45.72 0)
-    (effects (font (size 0.67 0.67)) (justify left bottom))
-  )
-  (text "AC712" (at 107.95 50.8 0)
-    (effects (font (size 0.62 0.62)) (justify left bottom))
-  )
-  (text "SDA" (at 74.295 72.39 0)
-    (effects (font (size 0.67 0.67)) (justify left bottom))
-  )
-  (text "AC_L" (at 83.82 55.88 0)
-    (effects (font (size 0.67 0.67)) (justify left bottom))
-  )
-  (label "D0" (at 34.29 38.735 0)
-    (effects (font (size 0.66 0.66)) (justify left bottom))
-  )
-  (label "AC712" (at 57.15 36.195 0)
-    (effects (font (size 0.66 0.66)) (justify left bottom))
-  )
-  (label "SCL" (at 57.785 41.275 0)
-    (effects (font (size 0.66 0.66)) (justify left bottom))
-  )
-  (label "SDA" (at 57.785 43.815 0)
-    (effects (font (size 0.66 0.66)) (justify left bottom))
-  )
-  (label "D0" (at 57.785 38.735 0)
+  (label "VCC" (at 74.295 77.47 0)
+    (effects (font (size 0.66 0.66)) (justify left bottom))
+  )
+  (label "DpSlp" (at 33.655 38.735 0)
+    (effects (font (size 0.66 0.66)) (justify left bottom))
+  )
+  (label "AC_N" (at 83.82 55.88 0)
+    (effects (font (size 0.66 0.66)) (justify left bottom))
+  )
+  (label "Data" (at 57.785 36.195 0)
+    (effects (font (size 0.66 0.66)) (justify left bottom))
+  )
+  (label "AanUit" (at 57.15 46.355 0)
+    (effects (font (size 0.66 0.66)) (justify left bottom))
+  )
+  (label "GND" (at 96.52 62.865 90)
+    (effects (font (size 0.66 0.66)) (justify left bottom))
+  )
+  (label "GND" (at 46.355 73.66 90)
+    (effects (font (size 0.66 0.66)) (justify left bottom))
+  )
+  (label "VCC" (at 96.52 22.86 90)
+    (effects (font (size 0.66 0.66)) (justify left bottom))
+  )
+  (label "Data" (at 107.95 50.8 0)
+    (effects (font (size 0.66 0.66)) (justify left bottom))
+  )
+  (label "VCC" (at 43.815 28.575 90)
+    (effects (font (size 0.66 0.66)) (justify left bottom))
+  )
+  (label "SCL" (at 58.42 41.275 0)
+    (effects (font (size 0.66 0.66)) (justify left bottom))
+  )
+  (label "DpSlp" (at 57.15 38.735 0)
+    (effects (font (size 0.66 0.66)) (justify left bottom))
+  )
+  (label "AanUit" (at 85.725 27.94 0)
+    (effects (font (size 0.66 0.66)) (justify left bottom))
+  )
+  (label "AC_L" (at 83.82 45.72 0)
+    (effects (font (size 0.66 0.66)) (justify left bottom))
+  )
+  (label "SCL" (at 74.295 74.93 0)
+    (effects (font (size 0.66 0.66)) (justify left bottom))
+  )
+  (label "SDA" (at 58.42 43.815 0)
+    (effects (font (size 0.66 0.66)) (justify left bottom))
+  )
+  (label "GND" (at 74.295 80.01 0)
+    (effects (font (size 0.66 0.66)) (justify left bottom))
+  )
+  (label "SDA" (at 74.295 72.39 0)
     (effects (font (size 0.66 0.66)) (justify left bottom))
   )
@@
       (effects (font (size 0.67 0.67)))
     )
-    (property "Value" "AC_Live" (id 1) (at 75.565 53.5615 0)
+    (property "Value" "AC_Neutral" (id 1) (at 75.565 53.5615 0)
       (effects (font (size 0.67 0.67)))
     )
@@
   )
   (symbol (lib_id "MCU_Module:WeMos_D1_mini") (at 46.355 48.895 0) (unit 1)
-    (in_bom yes) (on_board yes) (fields_autoplaced)
-    (property "Reference" "U1" (id 0) (at 48.3744 68.8245 0)
-      (effects (font (size 1.27 1.27)) (justify left))
-    )
-    (property "Value" "WeMos_D1_mini" (id 1) (at 48.3744 71.5996 0)
-      (effects (font (size 1.27 1.27)) (justify left))
+    (in_bom yes) (on_board yes)
+    (property "Reference" "U1" (id 0) (at 37.465 59.69 90)
+      (effects (font (size 1.16 1.16)) (justify left))
+    )
+    (property "Value" "WeMos_D1_mini" (id 1) (at 36.195 61.595 90)
+      (effects (font (size 0.66 0.66)) (justify left))
     )
     (property "Footprint" "Module:WEMOS_D1_mini_light" (id 2) (at 46.355 78.105 0)
@@
     )
     (path "/832faf4d-3bbe-48b0-b081-92cefd3c4e42"
-      (reference "J3") (unit 1) (value "AC_Live") (footprint "")
+      (reference "J3") (unit 1) (value "AC_Neutral") (footprint "")
     )
     (path "/6e417949-1c0b-4e2c-a1ca-2496c5b6d272"
