File: PCBs/StroomMeterACS712.kicad_sch (KiCad schematic)
At the start: 20 parts, among them J1 OLED1604, J2 ACS712, J3 PWR_5V_pin, J4 WS2812, J5 PWR_5V_jst, K1 SRD-03VDC-SL-C, Q1 BC547, Q2 BC547, SW1 btnAanUit, SW2 SW_SPDT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

Commit message: Bijgewerkt
Parts:
- added J?: Voeding_in, Connector_JST:JST_EH_B2B-EH-A_1x02_P2.50mm_Vertical, symbol Connector_Generic:Conn_01x02
- added PS?: HLK-PM01_220V, Converter_ACDC:Converter_ACDC_HiLink_HLK-PMxx, symbol Converter_ACDC:HLK-PM01
Connections:
- net GND: now also PS?.3 (-Vout)
- net VCC: now also PS?.4 (+Vout)
- new net: J?.1 (Pin_1), PS?.2 (AC/N)
- new net: J?.2 (Pin_2), PS?.1 (AC/L)
Other:
- moved on the sheet: SW2
Changed lines of the file:
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@@
+    (stroke (width 0) (type default) (color 0 0 0 0))
+  )
+  (wire (pts (xy 171.196 50.038) (xy 167.894 50.038))
     (stroke (width 0) (type default) (color 0 0 0 0))
   )
@@
     (stroke (width 0) (type default) (color 0 0 0 0))
   )
+  (wire (pts (xy 173.736 49.149) (xy 171.196 49.149))
+    (stroke (width 0) (type default) (color 0 0 0 0))
+  )
   (wire (pts (xy 122.682 51.308) (xy 122.682 53.34))
     (stroke (width 0) (type default) (color 0 0 0 0))
@@
     (stroke (width 0) (type default) (color 0 0 0 0))
   )
+  (wire (pts (xy 173.736 54.229) (xy 171.196 54.229))
+    (stroke (width 0) (type default) (color 0 0 0 0))
+  )
   (polyline (pts (xy 71.628 82.55) (xy 112.014 82.55))
     (stroke (width 0) (type default) (color 0 0 0 0))
   )
-  (polyline (pts (xy 206.248 61.468) (xy 156.464 61.468))
+  (polyline (pts (xy 206.248 64.135) (xy 156.464 64.135))
     (stroke (width 0) (type default) (color 0 0 0 0))
   )
@@
     (stroke (width 0) (type default) (color 0 0 0 0))
   )
-  (polyline (pts (xy 156.464 19.812) (xy 156.464 61.468))
+  (polyline (pts (xy 156.464 19.812) (xy 156.464 64.135))
     (stroke (width 0) (type default) (color 0 0 0 0))
   )
@@
     (stroke (width 0) (type default) (color 0 0 0 0))
   )
+  (wire (pts (xy 194.056 49.149) (xy 196.342 49.149))
+    (stroke (width 0) (type default) (color 0 0 0 0))
+  )
+  (wire (pts (xy 171.196 54.229) (xy 171.196 52.578))
+    (stroke (width 0) (type default) (color 0 0 0 0))
+  )
   (polyline (pts (xy 22.86 101.6) (xy 43.688 101.6))
     (stroke (width 0) (type default) (color 0 0 0 0))
@@
     (stroke (width 0) (type default) (color 0 0 0 0))
   )
+  (wire (pts (xy 171.196 49.149) (xy 171.196 50.038))
+    (stroke (width 0) (type default) (color 0 0 0 0))
+  )
   (polyline (pts (xy 43.688 101.6) (xy 43.688 85.598))
     (stroke (width 0) (type default) (color 0 0 0 0))
@@
     (stroke (width 0) (type default) (color 0 0 0 0))
   )
+  (wire (pts (xy 196.342 47.625) (xy 196.342 49.149))
+    (stroke (width 0) (type default) (color 0 0 0 0))
+  )
   (wire (pts (xy 58.42 39.37) (xy 55.88 39.37))
     (stroke (width 0) (type default) (color 0 0 0 0))
@@
     (stroke (width 0) (type default) (color 0 0 0 0))
   )
+  (wire (pts (xy 171.196 52.578) (xy 167.894 52.578))
+    (stroke (width 0) (type default) (color 0 0 0 0))
+  )
   (wire (pts (xy 103.124 110.109) (xy 103.124 108.839))
     (stroke (width 0) (type default) (color 0 0 0 0))
@@
     (stroke (width 0) (type default) (color 0 0 0 0))
   )
-  (polyline (pts (xy 206.248 19.812) (xy 206.248 61.468))
+  (polyline (pts (xy 206.248 19.812) (xy 206.248 64.135))
     (stroke (width 0) (type default) (color 0 0 0 0))
   )
@@
     (stroke (width 0) (type default) (color 0 0 0 0))
   )
+  (wire (pts (xy 196.469 54.229) (xy 196.469 55.626))
+    (stroke (width 0) (type default) (color 0 0 0 0))
+  )
   (wire (pts (xy 122.682 28.194) (xy 122.682 23.749))
     (stroke (width 0) (type default) (color 0 0 0 0))
@@
   )
   (wire (pts (xy 110.236 115.189) (xy 103.124 115.189))
+    (stroke (width 0) (type default) (color 0 0 0 0))
+  )
+  (wire (pts (xy 194.056 54.229) (xy 196.469 54.229))
     (stroke (width 0) (type default) (color 0 0 0 0))
   )
@@
     (pin "1")
   )
+  (symbol (lib_id "Connector_Generic:Conn_01x02") (at 162.814 52.578 180) (unit 1)
+    (in_bom yes) (on_board yes)
+    (property "Reference" "J?" (id 0) (at 162.814 46.228 0))
+    (property "Value" "Voeding_in" (id 1) (at 162.814 47.879 0)
+      (effects (font (size 0.66 0.66)))
+    )
+    (property "Footprint" "Connector_JST:JST_EH_B2B-EH-A_1x02_P2.50mm_Vertical" (id 2) (at 162.814 52.578 0)
+      (effects (font (size 1.27 1.27)) hide)
+    )
+    (property "Datasheet" "~" (id 3) (at 162.814 52.578 0)
+      (effects (font (size 1.27 1.27)) hide)
+    )
+    (pin "1")
+    (pin "2")
+  )
   (symbol (lib_id "Connector_Generic:Conn_01x02") (at 102.362 72.644 0) (unit 1)
     (in_bom yes) (on_board yes) (fields_autoplaced)
@@
     (pin "4")
     (pin "5")
+  )
+  (symbol (lib_name "GND_2") (lib_id "power:GND") (at 196.469 55.626 0) (unit 1)
+    (in_bom yes) (on_board yes)
+    (property "Reference" "#PWR?" (id 0) (at 196.469 61.976 0)
+      (effects (font (size 1.27 1.27)) hide)
+    )
+    (property "Value" "GND" (id 1) (at 196.596 59.436 0)
+      (effects (font (size 0.88 0.88)))
+    )
+    (property "Footprint" "" (id 2) (at 196.469 55.626 0)
+      (effects (font (size 1.27 1.27)) hide)
+    )
+    (property "Datasheet" "" (id 3) (at 196.469 55.626 0)
+      (effects (font (size 1.27 1.27)) hide)
+    )
+    (pin "1")
   )
   (symbol (lib_id "Device:R_Small_US") (at 112.268 112.649 90) (unit 1)
@@
     (pin "1")
   )
-  (symbol (lib_id "Switch:SW_SPDT") (at 175.006 53.975 0) (unit 1)
+  (symbol (lib_id "Converter_ACDC:HLK-PM01") (at 183.896 51.689 0) (unit 1)
+    (in_bom yes) (on_board yes)
+    (property "Reference" "PS?" (id 0) (at 183.515 44.577 0))
+    (property "Value" "HLK-PM01_220V" (id 1) (at 183.769 46.609 0)
+      (effects (font (size 0.8 0.8)))
+    )
+    (property "Footprint" "Converter_ACDC:Converter_ACDC_HiLink_HLK-PMxx" (id 2) (at 183.896 59.309 0)
+      (effects (font (size 1.27 1.27)) hide)
+    )
+    (property "Datasheet" "http://www.hlktech.net/product_detail.php?ProId=54" (id 3) (at 194.056 60.579 0)
+      (effects (font (size 1.27 1.27)) hide)
+    )
+    (pin "1")
+    (pin "2")
+    (pin "3")
+    (pin "4")
+  )
+  (symbol (lib_id "Switch:SW_SPDT") (at 198.374 29.591 0) (unit 1)
     (in_bom yes) (on_board yes) (fields_autoplaced)
-    (property "Reference" "SW2" (id 0) (at 175.006 47.371 0))
-    (property "Value" "SW_SPDT" (id 1) (at 175.006 49.911 0)
+    (property "Reference" "SW2" (id 0) (at 198.374 22.987 0))
+    (property "Value" "SW_SPDT" (id 1) (at 198.374 25.527 0)
       (effects (font (size 0.8 0.8)))
     )
-    (property "Footprint" "" (id 2) (at 175.006 53.975 0)
-      (effects (font (size 1.27 1.27)) hide)
-    )
-    (property "Datasheet" "~" (id 3) (at 175.006 53.975 0)
+    (property "Footprint" "" (id 2) (at 198.374 29.591 0)
+      (effects (font (size 1.27 1.27)) hide)
+    )
+    (property "Datasheet" "~" (id 3) (at 198.374 29.591 0)
       (effects (font (size 1.27 1.27)) hide)
     )
@@
     (pin "3")
   )
+  (symbol (lib_name "VCC_1") (lib_id "power:VCC") (at 196.342 47.625 0) (unit 1)
+    (in_bom yes) (on_board yes)
+    (property "Reference" "#PWR?" (id 0) (at 196.342 51.435 0)
+      (effects (font (size 1.27 1.27)) hide)
+    )
+    (property "Value" "VCC" (id 1) (at 196.342 43.942 0)
+      (effects (font (size 0.8 0.8)))
+    )
+    (property "Footprint" "" (id 2) (at 196.342 47.625 0)
+      (effects (font (size 1.27 1.27)) hide)
+    )
+    (property "Datasheet" "" (id 3) (at 196.342 47.625 0)
+      (effects (font (size 1.27 1.27)) hide)
+    )
+    (pin "1")
+  )
   (symbol (lib_id "power:GND") (at 122.682 53.34 0) (unit 1)
     (in_bom yes) (on_board yes)
@@
       (reference "#PWR0109") (unit 1) (value "VCC") (footprint "")
     )
+    (path "/31a064e3-adf7-4c9e-be7d-1193ce0579b1"
+      (reference "#PWR?") (unit 1) (value "GND") (footprint "")
+    )
+    (path "/f206b1a1-64e2-4364-bc14-b9085806ba7d"
+      (reference "#PWR?") (unit 1) (value "VCC") (footprint "")
+    )
     (path "/f8d28331-eeae-4d87-867f-0a521759c2f1"
       (reference "H1") (unit 1) (value "Gaatje") (footprint "MountingHole:MountingHole_2.7mm_M2.5_Pad")
@@
       (reference "J5") (unit 1) (value "PWR_5V_jst") (footprint "Connector_JST:JST_EH_B2B-EH-A_1x02_P2.50mm_Vertical")
     )
+    (path "/08f50ae6-9197-4cc7-bf93-a9c3e9cebd47"
+      (reference "J?") (unit 1) (value "Voeding_in") (footprint "Connector_JST:JST_EH_B2B-EH-A_1x02_P2.50mm_Vertical")
+    )
     (path "/2c38c161-17dc-4f92-b89f-4df0368010f6"
       (reference "K1") (unit 1) (value "SRD-03VDC-SL-C") (footprint "Relay_THT:Relay_SPDT_SANYOU_SRD_Series_Form_C")
     )
+    (path "/c2b2ae9d-9de9-41a3-a83b-7ea5a297950e"
+      (reference "PS?") (unit 1) (value "HLK-PM01_220V") (footprint "Converter_ACDC:Converter_ACDC_HiLink_HLK-PMxx")
+    )
     (path "/6e417949-1c0b-4e2c-a1ca-2496c5b6d272"

Commit message: Bijgewerkt
Parts:
- gave numbers to parts that had none: 2
Changed lines of the file:
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@@
   (symbol (lib_id "Connector_Generic:Conn_01x02") (at 162.814 52.578 180) (unit 1)
     (in_bom yes) (on_board yes)
-    (property "Reference" "J?" (id 0) (at 162.814 46.228 0))
+    (property "Reference" "J6" (id 0) (at 162.814 46.228 0))
     (property "Value" "Voeding_in" (id 1) (at 162.814 47.879 0)
       (effects (font (size 0.66 0.66)))
@@
   (symbol (lib_name "GND_2") (lib_id "power:GND") (at 196.469 55.626 0) (unit 1)
     (in_bom yes) (on_board yes)
-    (property "Reference" "#PWR?" (id 0) (at 196.469 61.976 0)
+    (property "Reference" "#PWR010" (id 0) (at 196.469 61.976 0)
       (effects (font (size 1.27 1.27)) hide)
     )
@@
   (symbol (lib_id "Converter_ACDC:HLK-PM01") (at 183.896 51.689 0) (unit 1)
     (in_bom yes) (on_board yes)
-    (property "Reference" "PS?" (id 0) (at 183.515 44.577 0))
+    (property "Reference" "PS1" (id 0) (at 183.515 44.577 0))
     (property "Value" "HLK-PM01_220V" (id 1) (at 183.769 46.609 0)
       (effects (font (size 0.8 0.8)))
@@
   (symbol (lib_name "VCC_1") (lib_id "power:VCC") (at 196.342 47.625 0) (unit 1)
     (in_bom yes) (on_board yes)
-    (property "Reference" "#PWR?" (id 0) (at 196.342 51.435 0)
+    (property "Reference" "#PWR09" (id 0) (at 196.342 51.435 0)
       (effects (font (size 1.27 1.27)) hide)
     )
@@
       (reference "#PWR08") (unit 1) (value "VCC") (footprint "")
     )
+    (path "/f206b1a1-64e2-4364-bc14-b9085806ba7d"
+      (reference "#PWR09") (unit 1) (value "VCC") (footprint "")
+    )
+    (path "/31a064e3-adf7-4c9e-be7d-1193ce0579b1"
+      (reference "#PWR010") (unit 1) (value "GND") (footprint "")
+    )
     (path "/5baaad51-90c9-47e6-8528-1e99fbd4fc0a"
       (reference "#PWR0101") (unit 1) (value "GND") (footprint "")
@@
       (reference "#PWR0109") (unit 1) (value "VCC") (footprint "")
     )
-    (path "/31a064e3-adf7-4c9e-be7d-1193ce0579b1"
-      (reference "#PWR?") (unit 1) (value "GND") (footprint "")
-    )
-    (path "/f206b1a1-64e2-4364-bc14-b9085806ba7d"
-      (reference "#PWR?") (unit 1) (value "VCC") (footprint "")
-    )
     (path "/f8d28331-eeae-4d87-867f-0a521759c2f1"
       (reference "H1") (unit 1) (value "Gaatje") (footprint "MountingHole:MountingHole_2.7mm_M2.5_Pad")
@@
     )
     (path "/08f50ae6-9197-4cc7-bf93-a9c3e9cebd47"
-      (reference "J?") (unit 1) (value "Voeding_in") (footprint "Connector_JST:JST_EH_B2B-EH-A_1x02_P2.50mm_Vertical")
+      (reference "J6") (unit 1) (value "Voeding_in") (footprint "Connector_JST:JST_EH_B2B-EH-A_1x02_P2.50mm_Vertical")
     )
     (path "/2c38c161-17dc-4f92-b89f-4df0368010f6"
@@
     )
     (path "/c2b2ae9d-9de9-41a3-a83b-7ea5a297950e"
-      (reference "PS?") (unit 1) (value "HLK-PM01_220V") (footprint "Converter_ACDC:Converter_ACDC_HiLink_HLK-PMxx")
+      (reference "PS1") (unit 1) (value "HLK-PM01_220V") (footprint "Converter_ACDC:Converter_ACDC_HiLink_HLK-PMxx")
     )
     (path "/6e417949-1c0b-4e2c-a1ca-2496c5b6d272"

Commit message: Bijgewerkt
Parts:
- J6: value Voeding_in -> 230V_in
- K1: value SRD-03VDC-SL-C -> SRD-03VDC-SL-C_Relay
Connections:
- net GND: now also K1.2
- net AC/L: now reaches J6.2 (Pin_2), PS1.1 (AC/L)
- net AC/L: now also K1.1, K1.4, SW2.2 (B)
Other:
- note added: "230V regeling"
- note removed: "220V Power regelaar"
- moved on the sheet: J6, K1, PS1, SW2
