File: PCBs/StroomMeterACS712.kicad_sch (KiCad schematic)
At the start: 22 parts, among them J1 OLED1604, J2 ACS712, J3 PWR_5V_pin, J4 WS2812, J5 PWR_5V_jst, J6 230V_in, K1 SRD-03VDC-SL-C_Relay, Q1 BC547, Q2 BC547, SW1 btnAanUit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

Commit message: PCF8574 toegevoegd aan PCB
Parts:
- R1: footprint Resistor_THT:R_Axial_DIN0204_L3.6mm_D1.6mm_P7.62mm_Horizontal -> Resistor_THT:R_Axial_DIN0204_L3.6mm_D1.6mm_P5.08mm_Horizontal
- R2, R3, R4: footprint (none) -> Resistor_THT:R_Axial_DIN0204_L3.6mm_D1.6mm_P5.08mm_Horizontal
- SW2: footprint (none) -> Button_Switch_THT:SW_PUSH_6mm
- U2: footprint (none) -> Package_DIP:DIP-16_W7.62mm
Changed lines of the file:
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@@
       (effects (font (size 0.66 0.66)))
     )
-    (property "Footprint" "" (id 2) (at 112.268 112.649 0)
+    (property "Footprint" "Resistor_THT:R_Axial_DIN0204_L3.6mm_D1.6mm_P5.08mm_Horizontal" (id 2) (at 112.268 112.649 0)
       (effects (font (size 1.27 1.27)) hide)
     )
@@
       (effects (font (size 0.66 0.66)))
     )
-    (property "Footprint" "" (id 2) (at 112.395 110.109 0)
+    (property "Footprint" "Resistor_THT:R_Axial_DIN0204_L3.6mm_D1.6mm_P5.08mm_Horizontal" (id 2) (at 112.395 110.109 0)
       (effects (font (size 1.27 1.27)) hide)
     )
@@
       (effects (font (size 0.66 0.66)))
     )
-    (property "Footprint" "" (id 2) (at 112.776 115.189 0)
+    (property "Footprint" "Resistor_THT:R_Axial_DIN0204_L3.6mm_D1.6mm_P5.08mm_Horizontal" (id 2) (at 112.776 115.189 0)
       (effects (font (size 1.27 1.27)) hide)
     )
@@
       (effects (font (size 1.27 1.27)) (justify left))
     )
-    (property "Footprint" "" (id 2) (at 133.096 112.649 0)
+    (property "Footprint" "Package_DIP:DIP-16_W7.62mm" (id 2) (at 133.096 112.649 0)
       (effects (font (size 1.27 1.27)) hide)
     )
@@
       (effects (font (size 0.8 0.8)))
     )
-    (property "Footprint" "" (id 2) (at 197.739 29.083 0)
+    (property "Footprint" "Button_Switch_THT:SW_PUSH_6mm" (id 2) (at 197.739 29.083 0)
       (effects (font (size 1.27 1.27)) hide)
     )
@@
       (effects (font (size 0.66 0.66)) (justify left))
     )
-    (property "Footprint" "Resistor_THT:R_Axial_DIN0204_L3.6mm_D1.6mm_P7.62mm_Horizontal" (id 2) (at 78.994 34.29 90)
+    (property "Footprint" "Resistor_THT:R_Axial_DIN0204_L3.6mm_D1.6mm_P5.08mm_Horizontal" (id 2) (at 78.994 34.29 90)
       (effects (font (size 1.27 1.27)) hide)
     )
@@
     )
     (path "/ff6377bc-0235-49a5-b06a-d57cc4533c3e"
-      (reference "R1") (unit 1) (value "R100") (footprint "Resistor_THT:R_Axial_DIN0204_L3.6mm_D1.6mm_P7.62mm_Horizontal")
+      (reference "R1") (unit 1) (value "R100") (footprint "Resistor_THT:R_Axial_DIN0204_L3.6mm_D1.6mm_P5.08mm_Horizontal")
     )
     (path "/417d3d17-b48f-4c16-a48d-0c48bb9d5e45"
-      (reference "R2") (unit 1) (value "R10K") (footprint "")
+      (reference "R2") (unit 1) (value "R10K") (footprint "Resistor_THT:R_Axial_DIN0204_L3.6mm_D1.6mm_P5.08mm_Horizontal")
     )
     (path "/61dd7ef3-b57a-4af3-911d-0a98fa833dee"
-      (reference "R3") (unit 1) (value "R10K") (footprint "")
+      (reference "R3") (unit 1) (value "R10K") (footprint "Resistor_THT:R_Axial_DIN0204_L3.6mm_D1.6mm_P5.08mm_Horizontal")
     )
     (path "/8da5da65-9db8-4bf8-9f57-2e1c669b2c30"
-      (reference "R4") (unit 1) (value "R10K") (footprint "")
+      (reference "R4") (unit 1) (value "R10K") (footprint "Resistor_THT:R_Axial_DIN0204_L3.6mm_D1.6mm_P5.08mm_Horizontal")
     )
     (path "/a4cdc196-e672-47ec-a411-7dd83efc16bb"
@@
     )
     (path "/c8685be6-5949-42cb-a590-5f7191490973"
-      (reference "SW2") (unit 1) (value "SW_SPDT") (footprint "")
+      (reference "SW2") (unit 1) (value "SW_SPDT") (footprint "Button_Switch_THT:SW_PUSH_6mm")
     )
     (path "/866c2804-79f0-42ad-b60b-35330f41683f"
@@
     )
     (path "/a2fb14b3-0721-4152-97d8-9d24afdd0b0d"
-      (reference "U2") (unit 1) (value "PCF8574A") (footprint "")
-    )
-  )
+      (reference "U2") (unit 1) (value "PCF8574A") (footprint "Package_DIP:DIP-16_W7.62mm")
+    )
+  )
