File: PCBs/StroomMeterACS712.kicad_pcb (KiCad board)
At the start: 2 copper layers, 22 parts, among them J1 OLED1604, J2 ACS712, J3 PWR_5V_pin, J4 WS2812, J5 PWR_5V_jst, J6 230V_in, K1 SRD-03VDC-SL-C_Relay, Q1 BC547, Q2 BC547, SW1 btnAanUit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

Commit message: autorouter toegevoegd
Connections:
- U2 pad 14: SDA -> SCL
- U2 pad 4: unconnected-(U2-Pad4) -> ACS_AanUit
Routing:
- net GND: track 0.00 -> 179.7 mm
- net VCC: track 0.00 -> 174.1 mm
- net SDA: track 0.00 -> 107.6 mm
- net AC/L: track 0.00 -> 59.3 mm
- net BTN1: track 0.00 -> 30.5 mm
- net ACS_AanUit: track 0.00 -> 29.2 mm
- net WS2812: track 0.00 -> 28.8 mm
- net Net-(J6-Pin_1): track 0.00 -> 24.2 mm
- net Net-(R1-Pad1): track 0.00 -> 21.9 mm
- net ACS_DATA: track 0.00 -> 17.9 mm
- net +5V: track 0.00 -> 17.6 mm
- net Net-(U2-A2): track 0.00 -> 11.0 mm
- net Net-(U2-A1): track 0.00 -> 10.0 mm
- net Net-(Q2-B): track 0.00 -> 9.88 mm
- net SCL: track 0.00 -> 8.81 mm
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Other:
- board text added: "/NC"
- board text added: "230V in GEVAAR!!!!"
- board text added: "AC-E"
- board text added: "AC-L"
- board text added: "ACS712"
- board text added: "BC547"
- board text added: "Data"
- board text added: "GND"
- board text added: "OLED1604"
- board text added: "PCF8574"
- board text added: "PWR_5V_jst"
- board text added: "R100"
- board text added: "R10K"
- board text added: "SCL"
- board text added: "SDA"
- board text added: "SRD-03VDC-SL-C_Relay"
- board text added: "SW_SPDT"
- board text added: "VCC"
- board text added: "WS2812"
- board text added: "btnAanUit"
