File: hardware/StroomMeterACS712.kicad_sch (KiCad schematic)
At the start: 6 parts, among them J2 AC_Live, J3 AC_Live, Q1 BC547, U1 WeMos_D1_mini, U2 ACS712xLCTR-05B

Commit message: bijgewerkt
Parts:
- added U?: PCF8574, symbol Interface_Expansion:PCF8574
Connections:
- net GND: now also U1.10 (GND)
- net VCC: now also U1.9 (5V)
- new net SCL: U?.14 (SCL)
- new net SDA: U?.15 (SDA)
- no-connect marks 5 -> 6
Changed lines of the file:
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@@
   (no_connect (at 33.02 46.99))
   (no_connect (at 55.88 49.53))
-  (no_connect (at 48.895 28.575))
+  (no_connect (at 71.12 127))
+  (no_connect (at 48.26 29.21))
   (no_connect (at 111.125 53.34))
   (bus_entry (at 59.69 44.45) (size 2.54 2.54)
@@
     (stroke (width 0) (type default) (color 0 0 0 0))
   )
+  (bus_entry (at 71.12 93.98) (size 2.54 2.54)
+    (stroke (width 0) (type default) (color 0 0 0 0))
+  )
+  (bus_entry (at 59.69 36.83) (size 2.54 2.54)
+    (stroke (width 0) (type default) (color 0 0 0 0))
+  )
+  (bus_entry (at 71.12 96.52) (size 2.54 2.54)
+    (stroke (width 0) (type default) (color 0 0 0 0))
+  )
   (bus_entry (at 59.69 46.99) (size 2.54 2.54)
     (stroke (width 0) (type default) (color 0 0 0 0))
@@
     (stroke (width 0) (type default) (color 0 0 0 0))
   )
-  (bus_entry (at 59.69 36.83) (size 2.54 2.54)
-    (stroke (width 0) (type default) (color 0 0 0 0))
-  )
   (bus_entry (at 71.12 77.47) (size 2.54 2.54)
     (stroke (width 0) (type default) (color 0 0 0 0))
@@
     (stroke (width 0) (type default) (color 0 0 0 0))
   )
-  (wire (pts (xy 41.275 24.765) (xy 43.815 24.765))
+  (wire (pts (xy 40.64 25.4) (xy 43.18 25.4))
+    (stroke (width 0) (type default) (color 0 0 0 0))
+  )
+  (wire (pts (xy 45.72 69.85) (xy 45.72 73.66))
+    (stroke (width 0) (type default) (color 0 0 0 0))
+  )
+  (wire (pts (xy 73.66 99.06) (xy 81.28 99.06))
     (stroke (width 0) (type default) (color 0 0 0 0))
   )
@@
     (stroke (width 0) (type default) (color 0 0 0 0))
   )
+  (bus (pts (xy 62.23 39.37) (xy 62.23 41.91))
+    (stroke (width 0) (type default) (color 0 0 0 0))
+  )
   (wire (pts (xy 73.66 80.01) (xy 76.835 80.01))
     (stroke (width 0) (type default) (color 0 0 0 0))
   )
+  (bus (pts (xy 71.12 96.52) (xy 71.12 127))
+    (stroke (width 0) (type default) (color 0 0 0 0))
+  )
   (wire (pts (xy 73.66 72.39) (xy 76.835 72.39))
     (stroke (width 0) (type default) (color 0 0 0 0))
   )
-  (bus (pts (xy 62.23 39.37) (xy 62.23 41.91))
-    (stroke (width 0) (type default) (color 0 0 0 0))
-  )
   (bus (pts (xy 71.12 74.93) (xy 71.12 77.47))
     (stroke (width 0) (type default) (color 0 0 0 0))
   )
+  (wire (pts (xy 55.88 36.83) (xy 59.69 36.83))
+    (stroke (width 0) (type default) (color 0 0 0 0))
+  )
   (wire (pts (xy 106.68 53.34) (xy 111.125 53.34))
     (stroke (width 0) (type default) (color 0 0 0 0))
   )
+  (bus (pts (xy 71.12 77.47) (xy 71.12 93.98))
+    (stroke (width 0) (type default) (color 0 0 0 0))
+  )
   (bus (pts (xy 71.12 64.77) (xy 71.12 69.85))
     (stroke (width 0) (type default) (color 0 0 0 0))
@@
     (stroke (width 0) (type default) (color 0 0 0 0))
   )
+  (bus (pts (xy 71.12 93.98) (xy 71.12 96.52))
+    (stroke (width 0) (type default) (color 0 0 0 0))
+  )
+  (wire (pts (xy 73.66 96.52) (xy 81.28 96.52))
+    (stroke (width 0) (type default) (color 0 0 0 0))
+  )
   (wire (pts (xy 33.02 46.99) (xy 35.56 46.99))
     (stroke (width 0) (type default) (color 0 0 0 0))
@@
     (stroke (width 0) (type default) (color 0 0 0 0))
   )
-  (wire (pts (xy 46.355 69.215) (xy 46.355 73.66))
-    (stroke (width 0) (type default) (color 0 0 0 0))
-  )
   (wire (pts (xy 55.88 39.37) (xy 59.69 39.37))
     (stroke (width 0) (type default) (color 0 0 0 0))
@@
     (stroke (width 0) (type default) (color 0 0 0 0))
   )
-  (wire (pts (xy 55.88 36.83) (xy 59.69 36.83))
-    (stroke (width 0) (type default) (color 0 0 0 0))
-  )
   (bus (pts (xy 71.12 72.39) (xy 71.12 74.93))
     (stroke (width 0) (type default) (color 0 0 0 0))
   )
-  (wire (pts (xy 43.815 28.575) (xy 43.815 24.765))
+  (wire (pts (xy 43.18 29.21) (xy 43.18 25.4))
     (stroke (width 0) (type default) (color 0 0 0 0))
   )
@@
     (effects (font (size 0.67 0.67)) (justify right bottom))
   )
-  (text "GND" (at 46.355 71.12 270)
+  (text "GND" (at 45.72 71.12 270)
     (effects (font (size 0.67 0.67)) (justify right bottom))
   )
@@
   (text "AC_L" (at 83.82 55.88 0)
     (effects (font (size 0.67 0.67)) (justify left bottom))
+  )
+  (label "SCL" (at 78.74 96.52 0)
+    (effects (font (size 0.66 0.66)) (justify left bottom))
+  )
+  (label "SDA" (at 78.74 99.06 0)
+    (effects (font (size 0.66 0.66)) (justify left bottom))
   )
   (symbol (lib_id "Sensor_Current:ACS712xLCTR-05B") (at 96.52 50.8 0) (unit 1)
@@
     (pin "1")
   )
-  (symbol (lib_id "power:GND") (at 46.355 73.66 0) (unit 1)
+  (symbol (lib_id "power:GND") (at 45.72 73.66 0) (unit 1)
     (in_bom yes) (on_board yes)
-    (property "Reference" "#PWR0101" (id 0) (at 46.355 80.01 0)
-      (effects (font (size 1.27 1.27)) hide)
-    )
-    (property "Value" "GND" (id 1) (at 45.085 76.835 0)
+    (property "Reference" "#PWR0101" (id 0) (at 45.72 80.01 0)
+      (effects (font (size 1.27 1.27)) hide)
+    )
+    (property "Value" "GND" (id 1) (at 44.45 76.835 0)
       (effects (font (size 0.67 0.67)) (justify left))
     )
-    (property "Footprint" "" (id 2) (at 46.355 73.66 0)
-      (effects (font (size 1.27 1.27)) hide)
-    )
-    (property "Datasheet" "" (id 3) (at 46.355 73.66 0)
+    (property "Footprint" "" (id 2) (at 45.72 73.66 0)
+      (effects (font (size 1.27 1.27)) hide)
+    )
+    (property "Datasheet" "" (id 3) (at 45.72 73.66 0)
       (effects (font (size 1.27 1.27)) hide)
     )
@@
     (pin "9")
   )
+  (symbol (lib_id "power:VCC") (at 40.64 25.4 90) (unit 1)
+    (in_bom yes) (on_board yes) (fields_autoplaced)
+    (property "Reference" "#PWR0104" (id 0) (at 44.45 25.4 0)
+      (effects (font (size 0.9 0.9)) hide)
+    )
+    (property "Value" "VCC" (id 1) (at 37.465 25.879 90)
+      (effects (font (size 0.66 0.66)) (justify left))
+    )
+    (property "Footprint" "" (id 2) (at 40.64 25.4 0)
+      (effects (font (size 1.27 1.27)) hide)
+    )
+    (property "Datasheet" "" (id 3) (at 40.64 25.4 0)
+      (effects (font (size 1.27 1.27)) hide)
+    )
+    (pin "1")
+  )
   (symbol (lib_id "Connector_Generic:Conn_01x01") (at 75.565 45.72 180) (unit 1)
     (in_bom yes) (on_board yes) (fields_autoplaced)
@@
     )
     (pin "1")
+  )
+  (symbol (lib_id "Interface_Expansion:PCF8574") (at 93.98 106.68 0) (unit 1)
+    (in_bom yes) (on_board yes) (fields_autoplaced)
+    (property "Reference" "U?" (id 0) (at 95.9994 87.4735 0)
+      (effects (font (size 1.27 1.27)) (justify left))
+    )
+    (property "Value" "PCF8574" (id 1) (at 95.9994 90.2486 0)
+      (effects (font (size 1.27 1.27)) (justify left))
+    )
+    (property "Footprint" "" (id 2) (at 93.98 106.68 0)
+      (effects (font (size 1.27 1.27)) hide)
+    )
+    (property "Datasheet" "http://www.nxp.com/documents/data_sheet/PCF8574_PCF8574A.pdf" (id 3) (at 93.98 106.68 0)
+      (effects (font (size 1.27 1.27)) hide)
+    )
+    (pin "1")
+    (pin "10")
+    (pin "11")
+    (pin "12")
+    (pin "13")
+    (pin "14")
+    (pin "15")
+    (pin "16")
+    (pin "2")
+    (pin "3")
+    (pin "4")
+    (pin "5")
+    (pin "6")
+    (pin "7")
+    (pin "8")
+    (pin "9")
   )
   (symbol (lib_id "Connector_Generic:Conn_01x04") (at 81.915 74.93 0) (unit 1)
@@
       (reference "#PWR0103") (unit 1) (value "GND") (footprint "")
     )
+    (path "/872bf435-c9d7-43c1-a1fc-da5ccd1e155d"
+      (reference "#PWR0104") (unit 1) (value "VCC") (footprint "")
+    )
     (path "/966fb941-502f-4c6f-9b0f-0c7b488134e8"
       (reference "J2") (unit 1) (value "AC_Live") (footprint "")
@@
       (reference "U2") (unit 1) (value "ACS712xLCTR-05B") (footprint "Package_SO:SOIC-8_3.9x4.9mm_P1.27mm")
     )
-  )
+    (path "/9eefbcc2-9746-4dc8-a009-c9898547d9a9"
+      (reference "U?") (unit 1) (value "PCF8574") (footprint "")
+    )
+  )
